Commit message: Added robot class for management of robot operations. Added force topic for robot commands with gazebo

File: src/panda_world/models/panda/panda.urdf (robot description, URDF)
Before this commit: robot fp3, 15 links, 14 joints
Joints:
- joint fp3_finger_joint1: type prismatic -> fixed
- joint fp3_finger_joint2: mimic joint=fp3_finger_joint1 -> (none); type prismatic -> fixed
