Commit message: Added (wrong) ft sensors and camera

File: src/panda_world/models/panda/panda_fr3.urdf (robot description, URDF)
Before this commit: robot fr3, 14 links, 13 joints
Joints:
- joint world_joint: origin xyz=0 0 0 rpy=0 0 0 -> xyz=0 0 0.75 rpy=0 0 0

Commit message: Implemented cartesian trajectory with orientation trajectory generation

File: src/panda_world/models/panda/panda_fr3.urdf (robot description, URDF)
Before this commit: robot fr3, 14 links, 13 joints
Joints:
- joint fr3_joint1: limit lower=-2.7437 upper=2.7437 effort=87.0 velocity=2.62 -> lower=-2.8973 upper=2.8973 effort=87.0 velocity=2.1750
- joint fr3_joint2: limit lower=-1.7837 upper=1.7837 effort=87.0 velocity=2.62 -> lower=-1.7628 upper=1.7628 effort=87.0 velocity=2.1750
- joint fr3_joint3: limit lower=-2.9007 upper=2.9007 effort=87.0 velocity=2.62 -> lower=-2.8973 upper=2.8973 effort=87.0 velocity=2.1750
- joint fr3_joint4: limit lower=-3.0421 upper=-0.1518 effort=87.0 velocity=2.62 -> lower=-3.0718 upper=-0.0698 effort=87.0 velocity=2.1750
- joint fr3_joint5: limit lower=-2.8065 upper=2.8065 effort=12.0 velocity=5.26 -> lower=-2.8973 upper=2.8973 effort=12.0 velocity=2.6100
- joint fr3_joint6: limit lower=0.5445 upper=4.5169 effort=12.0 velocity=4.18 -> lower=-0.0175 upper=3.7525 effort=12.0 velocity=2.6100
- joint fr3_joint7: limit lower=-3.0159 upper=3.0159 effort=12.0 velocity=5.26 -> lower=-2.8973 upper=2.8973 effort=12.0 velocity=2.6100
