Commit message: Impelemented impedance controller with cartesian trajectory example

File: src/panda_world/models/panda/panda_fr3_no_table.urdf (robot description, URDF)
Before this commit: robot fr3, 13 links, 12 joints
Links:
- removed link fr3_hand
- removed link fr3_hand_tcp
- removed link fr3_leftfinger
- removed link fr3_link8
- removed link fr3_rightfinger
Joints:
- removed joint fr3_finger_joint1
- removed joint fr3_finger_joint2
- removed joint fr3_hand_joint
- removed joint fr3_hand_tcp_joint
- removed joint fr3_joint8
